Commit message: 09/27/2026 progress (forgot to track)

File: isaac_sim/robots/V1_Robot.urdf (robot description, URDF)
Before this commit: robot asn_robot, 6 links, 5 joints
Links:
- removed link laser_frame
- added link world
- link base_link: mass None -> 2.54999971; geometry collision cylinder length=0.0599999987 radius=0.164000005; collision mesh filename=./meshes/mesh_1_3.obj
Joints:
- removed joint base_to_laser
- added joint floating_base: type floating, parent world, child base_link
- joint left_wheel_joint: limit effort=3.40282347e+38 velocity=0.1 -> effort=3.40282347e+38
- joint right_wheel_joint: limit effort=3.40282347e+38 velocity=0.1 -> effort=3.40282347e+38
- joint wheel_drop_left_joint: limit lower=0 upper=0.0299999993 effort=3.40282347e+38 velocity=0.1 -> lower=0 upper=0.0299999993 effort=3.40282347e+38
- joint wheel_drop_right_joint: limit lower=0 upper=0.0299999993 effort=3.40282347e+38 velocity=0.1 -> lower=0 upper=0.0299999993 effort=3.40282347e+38
