Commit message: V3 Implementation Semantical Navigation -> Coverage Map

File: ros2_ws/src/asn_description/urdf/robot.urdf (robot description, URDF)
Before this commit: robot asn_robot, 6 links, 5 joints
Links:
- added link camera_link
- added link camera_optical_frame
Joints:
- added joint base_to_camera_link: type fixed, parent base_link, child camera_link, origin xyz=0 0 0.3 rpy=0 0 0
- added joint camera_link_to_camera_frame: type fixed, parent camera_link, child camera_optical_frame, origin xyz=0 0 0 rpy=-1.570796 0 -1.570796
